Commit message: Created URDF for Swerve Drive
Tank Drive will be unusable in simulation because those lines of code were commented out and replaced with the swerve. A separate URDF will probably be used later and either tank drive or serve drive will be selectable in the launch files.

File: catkin_ws/src/frc_robot/urdf/00-default.urdf (robot description, URDF)
Before this commit: robot myfirst, 17 links, 16 joints
Links:
- removed link fl_wheel
- removed link fr_wheel
- removed link ml_wheel
- removed link mr_wheel
- removed link rl_wheel
- removed link rr_wheel
- added link fl_swerve_pivot
- added link fl_swerve_wheel, mass 1; collision cylinder length=0.0381 radius=0.1016; visual cylinder length=0.0381 radius=0.1016
- added link fr_swerve_pivot
- added link fr_swerve_wheel, mass 1; collision cylinder length=0.0381 radius=0.1016; visual cylinder length=0.0381 radius=0.1016
- added link rl_swerve_pivot
- added link rl_swerve_wheel, mass 1; collision cylinder length=0.0381 radius=0.1016; visual cylinder length=0.0381 radius=0.1016
- added link rr_swerve_pivot
- added link rr_swerve_wheel, mass 1; collision cylinder length=0.0381 radius=0.1016; visual cylinder length=0.0381 radius=0.1016
Joints:
- removed joint base_link_to_fl_wheel
- removed joint base_link_to_fr_wheel
- removed joint base_link_to_ml_wheel
- removed joint base_link_to_mr_wheel
- removed joint base_link_to_rl_wheel
- removed joint base_link_to_rr_wheel
- added joint base_link_to_fl_swerve_pivot: type continuous, parent base_link, child fl_swerve_pivot, origin xyz=0.3048 0.3048 0.0 rpy=0 0 0, axis 0 0 1
- added joint base_link_to_fr_swerve_pivot: type continuous, parent base_link, child fr_swerve_pivot, origin xyz=0.3048 -0.3048 0.0 rpy=0 0 0, axis 0 0 1
- added joint base_link_to_rl_swerve_pivot: type continuous, parent base_link, child rl_swerve_pivot, origin xyz=-0.3048 0.3048 0.0 rpy=0 0 0, axis 0 0 1
- added joint base_link_to_rr_swerve_pivot: type continuous, parent base_link, child rr_swerve_pivot, origin xyz=-0.3048 -0.3048 0.0 rpy=0 0 0, axis 0 0 1
- added joint fl_swerve_pivot_to_fl_swerve_wheel: type continuous, parent fl_swerve_pivot, child fl_swerve_wheel, origin xyz=0 0 0 rpy=-1.57079632679 0 0, axis 0 0 1
- added joint fr_swerve_pivot_to_fr_swerve_wheel: type continuous, parent fr_swerve_pivot, child fr_swerve_wheel, origin xyz=0 0 0 rpy=-1.57079632679 0 0, axis 0 0 1
- added joint rl_swerve_pivot_to_rl_swerve_wheel: type continuous, parent rl_swerve_pivot, child rl_swerve_wheel, origin xyz=0 0 0 rpy=-1.57079632679 0 0, axis 0 0 1
- added joint rr_swerve_pivot_to_rr_swerve_wheel: type continuous, parent rr_swerve_pivot, child rr_swerve_wheel, origin xyz=0 0 0 rpy=-1.57079632679 0 0, axis 0 0 1

File: catkin_ws/src/frc_robot/urdf/00-default.urdf.xacro (robot description, xacro)
@@ -15,7 +15,10 @@
     chassis_length="0.8128" chassis_width="0.7112"
     chassis_height="0.1524" chassis_mass="50" />
-  <xacro:six_wheel_diff_drive name="tank_drive" parent="base_link"
+  <!-- <xacro:six_wheel_diff_drive name="tank_drive" parent="base_link"
     z_offset="0.0" drop_wheel_height="0.003175"
-    wheel_separation="0.6096" wheel_base_length="0.6096"
+    wheel_separation="0.6096" wheelbase_length="0.6096"
+    wheel_radius="0.1016" wheel_width="0.0381" wheel_mass="1" /> -->
+  <xacro:swerve_drive name="swerve_drive" parent="base_link"
+    z_offset="0.0" wheelbase_width="0.6096" wheelbase_length="0.6096"
     wheel_radius="0.1016" wheel_width="0.0381" wheel_mass="1" />
   <!-- <xacro:elevator_attachment name="elevator" parent="base_link"

File: catkin_ws/src/frc_robot/urdf/drivetrain.urdf.xacro (robot description, xacro)
@@ -10,9 +10,10 @@
       <xacro:property name="drop" value="-1" />
       <xacro:property name="high_friction" value="200.0" />
+      <xacro:property name="medium_friction" value="100.0" />
       <xacro:property name="low_friction" value="1.0" />
-    <xacro:macro name="six_wheel_diff_drive" params="name parent z_offset drop_wheel_height wheel_separation wheel_base_length wheel_radius wheel_width wheel_mass">
-    <!--                          Wheels                           -->
-      <xacro:macro name="wheel" params="prefix side fntctrbck drop friction">
-        <link name="${prefix}_wheel">
+    <xacro:macro name="six_wheel_diff_drive" params="name parent z_offset drop_wheel_height wheel_separation wheelbase_length wheel_radius wheel_width wheel_mass">
+    <!--                          Diff Wheels                           -->
+      <xacro:macro name="diff_wheel" params=" parent2 prefix side fntctrbck drop friction">
+        <link name="${prefix}_diff_wheel">
           <visual>
             <geometry>
@@ -37,20 +38,20 @@
           </inertial>
         </link>
-        <joint name="${parent}_to_${prefix}_wheel" type="continuous">
-          <parent link="${parent}"/>
-          <child link="${prefix}_wheel"/>
+        <joint name="${parent2}_to_${prefix}_diff_wheel" type="continuous">
+          <parent link="${parent2}"/>
+          <child link="${prefix}_diff_wheel"/>
           <axis xyz="0 0 ${-1*side}"/>
-          <origin rpy="${side*pi/2} 0 0" xyz="${fntctrbck*(wheel_base_length/2)} ${side*(wheel_separation/2)} ${z_offset+drop*drop_wheel_height}"/>
+          <origin rpy="${side*pi/2} 0 0" xyz="${fntctrbck*(wheelbase_length/2)} ${side*(wheel_separation/2)} ${z_offset+drop*drop_wheel_height}"/>
         </joint>
-        <transmission name="${prefix}_wheel_trans">
+        <transmission name="${prefix}_diff_wheel_trans">
           <type>transmission_interface/SimpleTransmission</type>
-          <actuator name="${prefix}_wheel_motor">
+          <actuator name="${prefix}_diff_wheel_motor">
             <mechanicalReduction>1</mechanicalReduction>
           </actuator>
-          <joint name="${parent}_to_${prefix}_wheel">
+          <joint name="${parent2}_to_${prefix}_diff_wheel">
             <hardwareInterface>hardware_interface/VelocityJointInterface</hardwareInterface>
           </joint>
         </transmission>
-        <gazebo reference="${prefix}_wheel">
+        <gazebo reference="${prefix}_diff_wheel">
           <mu1 value="${friction}"/>
           <mu2 value="${friction}"/>
@@ -60,10 +61,91 @@
         </gazebo>
       </xacro:macro>
-      <xacro:wheel prefix="fl" side="${left}" fntctrbck="${front}" drop="${no_drop}" friction="${low_friction}" />
-      <xacro:wheel prefix="ml" side="${left}" fntctrbck="${middle}" drop="${drop}" friction="${high_friction}" />
-      <xacro:wheel prefix="rl" side="${left}" fntctrbck="${rear}" drop="${no_drop}" friction="${low_friction}" />
-      <xacro:wheel prefix="fr" side="${right}" fntctrbck="${front}" drop="${no_drop}" friction="${low_friction}" />
-      <xacro:wheel prefix="mr" side="${right}" fntctrbck="${middle}" drop="${drop}" friction="${high_friction}" />
-      <xacro:wheel prefix="rr" side="${right}" fntctrbck="${rear}" drop="${no_drop}" friction="${low_friction}" />
+      <xacro:diff_wheel parent2="${parent}" prefix="fl" side="${left}" fntctrbck="${front}" drop="${no_drop}" friction="${low_friction}" />
+      <xacro:diff_wheel parent2="${parent}" prefix="ml" side="${left}" fntctrbck="${middle}" drop="${drop}" friction="${high_friction}" />
+      <xacro:diff_wheel parent2="${parent}" prefix="rl" side="${left}" fntctrbck="${rear}" drop="${no_drop}" friction="${low_friction}" />
+      <xacro:diff_wheel parent2="${parent}" prefix="fr" side="${right}" fntctrbck="${front}" drop="${no_drop}" friction="${low_friction}" />
+      <xacro:diff_wheel parent2="${parent}" prefix="mr" side="${right}" fntctrbck="${middle}" drop="${drop}" friction="${high_friction}" />
+      <xacro:diff_wheel parent2="${parent}" prefix="rr" side="${right}" fntctrbck="${rear}" drop="${no_drop}" friction="${low_friction}" />
+    </xacro:macro>
+    <xacro:macro name="swerve_drive" params="name parent z_offset wheelbase_width wheelbase_length wheel_radius wheel_width wheel_mass">
+    <!--                          Swerve Pivot                           -->
+      <xacro:macro name="swerve_pivot" params="parent2 prefix side fntbck friction">
+        <!--                          Swerve Wheel                           -->
+          <xacro:macro name="swerve_wheel" params="parent3 prefix2 friction">
+            <link name="${prefix2}_swerve_wheel">
+              <visual>
+                <geometry>
+                  <cylinder length="${wheel_width}" radius="${wheel_radius}"/>
+                </geometry>
+                <origin xyz="0 0 0"/>
+                <material name="blue"/>
+              </visual>
+              <collision>
+                <geometry>
+                  <cylinder length="${wheel_width}" radius="${wheel_radius}"/>
+                </geometry>
+                <origin xyz="0 0 0"/>
+              </collision>
+              <inertial>
+                <mass value="${wheel_mass}"/>
+                <xacro:cylinder_inertia
+                m="${wheel_mass}"
+                r="${wheel_radius}"
+                h="${wheel_width}" />
+                <origin xyz="0 0 0"/>
+              </inertial>
+            </link>
+            <joint name="${parent3}_to_${prefix2}_swerve_wheel" type="continuous">
+              <parent link="${parent3}"/>
+              <child link="${prefix2}_swerve_wheel"/>
+              <axis xyz="0 0 1"/>
+              <origin rpy="${-pi/2} 0 0" xyz="0 0 0"/>
+            </joint>
+            <transmission name="${prefix2}_swerve_wheel_trans">
+              <type>transmission_interface/SimpleTransmission</type>
+              <actuator name="${prefix2}_swerve_wheel_motor">
+                <mechanicalReduction>1</mechanicalReduction>
+              </actuator>
+              <joint name="${parent3}_to_${prefix2}_swerve_wheel">
+                <hardwareInterface>hardware_interface/VelocityJointInterface</hardwareInterface>
+              </joint>
+            </transmission>
+            <gazebo reference="${prefix2}_swerve_wheel">
+              <mu1 value="${friction}"/>
+              <mu2 value="${friction}"/>
+              <kp value="10000000.0"/>
+              <kd value="1.0" />
+              <material>Gazebo/gray</material>
+            </gazebo>
+          </xacro:macro>
+        <link name="${prefix}_swerve_pivot"/>
+        <joint name="${parent2}_to_${prefix}_swerve_pivot" type="continuous">
+          <parent link="${parent2}"/>
+          <child link="${prefix}_swerve_pivot"/>
+          <axis xyz="0 0 1"/>
+          <origin rpy="0 0 0" xyz="${fntbck*(wheelbase_length/2)} ${side*(wheelbase_width/2)} ${z_offset}"/>
+        </joint>
+        <xacro:swerve_wheel parent3="${prefix}_swerve_pivot" prefix2="${prefix}" friction="${friction}" />
+        <transmission name="${prefix}_swerve_pivot_trans">
+          <type>transmission_interface/SimpleTransmission</type>
+          <actuator name="${prefix}_swerve_pivot_motor">
+            <mechanicalReduction>1</mechanicalReduction>
+          </actuator>
+          <joint name="${parent2}_to_${prefix}_swerve_pivot">
+            <hardwareInterface>hardware_interface/PositionJointInterface</hardwareInterface>
+          </joint>
+        </transmission>
+        <gazebo reference="${prefix}_swerve_pivot">
+          <mu1 value="${friction}"/>
+          <mu2 value="${friction}"/>
+          <kp value="10000000.0"/>
+          <kd value="1.0" />
+          <material>Gazebo/gray</material>
+        </gazebo>
+      </xacro:macro>
+      <xacro:swerve_pivot parent2="${parent}" prefix="fl" side="${left}" fntbck="${front}" friction="${medium_friction}" />
+      <xacro:swerve_pivot parent2="${parent}" prefix="rl" side="${left}" fntbck="${rear}" friction="${medium_friction}" />
+      <xacro:swerve_pivot parent2="${parent}" prefix="fr" side="${right}" fntbck="${front}" friction="${medium_friction}" />
+      <xacro:swerve_pivot parent2="${parent}" prefix="rr" side="${right}" fntbck="${rear}" friction="${medium_friction}" />
   </xacro:macro>
 </root>

Commit message: Literally 3 weeks of work didn't get uploaded properly.
Dafuq? I'm not repeating all those updates.

File: catkin_ws/src/frc_robot/urdf/00-default.urdf (robot description, URDF)
Before this commit: robot myfirst, 19 links, 18 joints
Links:
- added link laser
- link fl_swerve_pivot: mass None -> 1.0; geometry collision cylinder length=0.1 radius=0.05; visual cylinder length=0.1 radius=0.05
- link fr_swerve_pivot: mass None -> 1.0; geometry collision cylinder length=0.1 radius=0.05; visual cylinder length=0.1 radius=0.05
- link rl_swerve_pivot: mass None -> 1.0; geometry collision cylinder length=0.1 radius=0.05; visual cylinder length=0.1 radius=0.05
- link rr_swerve_pivot: mass None -> 1.0; geometry collision cylinder length=0.1 radius=0.05; visual cylinder length=0.1 radius=0.05
Joints:
- removed joint base_link_to_lidar_mount
- added joint kinect_mount_to_camera_link: type fixed, parent kinect_mount, child camera_link, origin xyz=0 0 0 rpy=0 0 0
- added joint kinect_mount_to_lidar_mount: type fixed, parent kinect_mount, child lidar_mount, origin xyz=0 0 0.1 rpy=0 0 0
- added joint lidar_mount_to_laser: type fixed, parent lidar_mount, child laser, origin xyz=0 0 0 rpy=0 0 3.14159265359
- joint base_link_to_kinect_mount: origin xyz=0.25 0 0.5 rpy=0 0 0 -> xyz=0.25 0 0.2 rpy=0 0 0

File: catkin_ws/src/frc_robot/urdf/00-default.urdf.xacro (robot description, xacro)
@@ -29,11 +29,22 @@
     <parent link="base_link"/>
     <child link="kinect_mount"/>
-    <origin rpy="0 0 0" xyz="0.25 0 0.5"/>
+    <origin rpy="0 0 0" xyz="0.25 0 0.2"/>
   </joint>
   <link name="lidar_mount"/>
-  <joint name="base_link_to_lidar_mount" type="fixed">
-    <parent link="base_link"/>
+  <joint name="kinect_mount_to_lidar_mount" type="fixed">
+    <parent link="kinect_mount"/>
     <child link="lidar_mount"/>
-    <origin rpy="0 0 0" xyz="0.25 0 0.3"/>
+    <origin rpy="0 0 0" xyz="0 0 0.1"/>
+  </joint>
+  <joint name="kinect_mount_to_camera_link" type="fixed">
+    <parent link="kinect_mount"/>
+    <child link="camera_link"/>
+    <origin rpy="0 0 0" xyz="0 0 0"/>
+  </joint>
+  <link name="laser"/>
+  <joint name="lidar_mount_to_laser" type="fixed">
+    <parent link="lidar_mount"/>
+    <child link="laser"/>
+    <origin rpy="0 0 ${pi}" xyz="0 0 0"/>
   </joint>
   <xacro:sensor_kinect parent="kinect_mount"/>
@@ -54,5 +65,5 @@
   <gazebo>
     <plugin name="gazebo_ros_control" filename="libgazebo_ros_control.so">
-      <robotNamespace>/</robotNamespace>
+      <robotNamespace>/drivetrain</robotNamespace>
       <legacyModeNS>true</legacyModeNS>
     </plugin>

File: catkin_ws/src/frc_robot/urdf/drivetrain.urdf.xacro (robot description, xacro)
@@ -72,5 +72,5 @@
       <xacro:macro name="swerve_pivot" params="parent2 prefix side fntbck friction">
         <!--                          Swerve Wheel                           -->
-          <xacro:macro name="swerve_wheel" params="parent3 prefix2 friction">
+          <xacro:macro name="swerve_wheel" params="parent3 prefix2 friction2">
             <link name="${prefix2}_swerve_wheel">
               <visual>
@@ -105,4 +105,5 @@
               <type>transmission_interface/SimpleTransmission</type>
               <actuator name="${prefix2}_swerve_wheel_motor">
+                <hardwareInterface>hardware_interface/VelocityJointInterface</hardwareInterface>
                 <mechanicalReduction>1</mechanicalReduction>
               </actuator>
@@ -112,6 +113,6 @@
             </transmission>
             <gazebo reference="${prefix2}_swerve_wheel">
-              <mu1 value="${friction}"/>
-              <mu2 value="${friction}"/>
+              <mu1 value="${friction2}"/>
+              <mu2 value="${friction2}"/>
               <kp value="10000000.0"/>
               <kd value="1.0" />
@@ -119,15 +120,37 @@
             </gazebo>
           </xacro:macro>
-        <link name="${prefix}_swerve_pivot"/>
+        <link name="${prefix}_swerve_pivot">
+              <visual>
+                <geometry>
+                  <cylinder length="0.1" radius="0.05"/>
+                </geometry>
+                <origin xyz="0 0 0"/>
+                <material name="blue"/>
+              </visual>
+              <collision>
+                <geometry>
+                  <cylinder length="0.1" radius="0.05"/>
+                </geometry>
+                <origin xyz="0 0 0"/>
+              </collision>
+              <inertial>
+                <mass value="1.0"/>
+                <xacro:cylinder_inertia
+                m="1.0"
+                r="0.05"
+                h="0.1" />
+                <origin xyz="0 0 0"/>
+              </inertial>
+        </link>
         <joint name="${parent2}_to_${prefix}_swerve_pivot" type="continuous">
-          <parent link="${parent2}"/>
-          <child link="${prefix}_swerve_pivot"/>
-          <axis xyz="0 0 1"/>
-          <origin rpy="0 0 0" xyz="${fntbck*(wheelbase_length/2)} ${side*(wheelbase_width/2)} ${z_offset}"/>
+            <parent link="${parent2}"/>
+            <child link="${prefix}_swerve_pivot"/>
+            <axis xyz="0 0 1"/>
+            <origin rpy="0 0 0" xyz="${fntbck*(wheelbase_length/2)} ${side*(wheelbase_width/2)} ${z_offset}"/>
         </joint>
-        <xacro:swerve_wheel parent3="${prefix}_swerve_pivot" prefix2="${prefix}" friction="${friction}" />
         <transmission name="${prefix}_swerve_pivot_trans">
           <type>transmission_interface/SimpleTransmission</type>
           <actuator name="${prefix}_swerve_pivot_motor">
+            <hardwareInterface>hardware_interface/PositionJointInterface</hardwareInterface>
             <mechanicalReduction>1</mechanicalReduction>
           </actuator>
@@ -143,4 +166,5 @@
           <material>Gazebo/gray</material>
         </gazebo>
+        <xacro:swerve_wheel parent3="${prefix}_swerve_pivot" prefix2="${prefix}" friction2="${friction}" />
       </xacro:macro>
       <xacro:swerve_pivot parent2="${parent}" prefix="fl" side="${left}" fntbck="${front}" friction="${medium_friction}" />
