Commit message: Created branch to start hardware testing
Made new file for just using the kinect and lidar. Need to work on SLAM without wheel odometry while the actual robot is still unavailable.

File: catkin_ws/src/frc_robot/urdf/00-default.urdf.xacro (robot description, xacro)
@@ -26,5 +26,5 @@
     <parent link="base_link"/>
     <child link="kinect_mount"/>
-    <origin rpy="0 0 0" xyz="0.25 0 0.5"/>
+    <origin rpy="0 0 0" xyz="0.25 0 0.2"/>
   </joint>
   <link name="lidar_mount"/>
@@ -33,4 +33,16 @@
     <child link="lidar_mount"/>
     <origin rpy="0 0 0" xyz="0.25 0 0.3"/>
+  </joint>
+  <!-- <link name="camera_link"/> -->
+  <joint name="kinect_mount_to_camera_link" type="fixed">
+    <parent link="kinect_mount"/>
+    <child link="camera_link"/>
+    <origin rpy="0 0 0" xyz="0 0 0"/>
+  </joint>
+  <link name="laser"/>
+  <joint name="lidar_mount_to_laser" type="fixed">
+    <parent link="lidar_mount"/>
+    <child link="laser"/>
+    <origin rpy="0 0 ${pi}" xyz="0 0 0"/>
   </joint>
   <xacro:sensor_kinect parent="kinect_mount"/>

Commit message: Testing Hardware, setting up for no-ODOM SLAM.
Hardware is being tested, and the topics need to be consistent between sim and hardware. Also without the robot sending odometry, there needs to be a way to test SLAM without it.

File: catkin_ws/src/frc_robot/urdf/00-default.urdf.xacro (robot description, xacro)
@@ -29,10 +29,9 @@
   </joint>
   <link name="lidar_mount"/>
-  <joint name="base_link_to_lidar_mount" type="fixed">
-    <parent link="base_link"/>
+  <joint name="kinect_mount_to_lidar_mount" type="fixed">
+    <parent link="kinect_mount"/>
     <child link="lidar_mount"/>
-    <origin rpy="0 0 0" xyz="0.25 0 0.3"/>
+    <origin rpy="0 0 0" xyz="0 0 0.1"/>
   </joint>
-  <!-- <link name="camera_link"/> -->
   <joint name="kinect_mount_to_camera_link" type="fixed">
     <parent link="kinect_mount"/>

Commit message: Modifying urdf. Pivot joints dont work.

File: catkin_ws/src/frc_robot/urdf/00-default.urdf.xacro (robot description, xacro)
@@ -21,5 +21,5 @@
   <xacro:swerve_drive name="swerve_drive" parent="base_link"
     z_offset="0.0" wheelbase_width="0.6096" wheelbase_length="0.6096"
-    wheel_radius="0.1016" wheel_width="0.0381" wheel_mass="1" />
+    wheel_radius="0.03175" wheel_width="0.0381" wheel_mass="1" />
   <!-- <xacro:elevator_attachment name="elevator" parent="base_link"
     ax="0.0" ay="0.0" az="0.0762" rr="0.0" rp="0.0" ry="0.0"/> -->

File: catkin_ws/src/frc_robot/urdf/drivetrain.urdf.xacro (robot description, xacro)
@@ -12,4 +12,7 @@
       <xacro:property name="medium_friction" value="100.0" />
       <xacro:property name="low_friction" value="1.0" />
+      <xacro:property name="pivot_radius" value="0.025" />
+      <xacro:property name="pivot_height" value="0.025" />
+      <xacro:property name="pivot_mass" value="1.0" />
     <xacro:macro name="six_wheel_diff_drive" params="name parent z_offset drop_wheel_height wheel_separation wheelbase_length wheel_radius wheel_width wheel_mass">
     <!--                          Diff Wheels                           -->
@@ -123,22 +126,22 @@
               <visual>
                 <geometry>
-                  <cylinder length="0.1" radius="0.05"/>
+                  <cylinder length="${pivot_height}" radius="${pivot_radius}"/>
                 </geometry>
-                <origin xyz="0 0 0"/>
+                <origin xyz="0 0 ${pivot_height/2}"/>
                 <material name="blue"/>
               </visual>
               <collision>
                 <geometry>
-                  <cylinder length="0.1" radius="0.05"/>
+                  <cylinder length="${pivot_height}" radius="${pivot_radius}"/>
                 </geometry>
-                <origin xyz="0 0 0"/>
+                <origin xyz="0 0 ${pivot_height/2}"/>
               </collision>
               <inertial>
-                <mass value="1.0"/>
+                <mass value="${pivot_mass}"/>
                 <xacro:cylinder_inertia
-                m="1.0"
-                r="0.05"
-                h="0.1" />
-                <origin xyz="0 0 0"/>
+                m="${pivot_mass}"
+                r="${pivot_radius}"
+                h="${pivot_height}" />
+                <origin xyz="0 0 ${pivot_height/2}"/>
               </inertial>
         </link>

Commit message: Major localization overhaul.
Wheel and IMU-only ODOM works very well. Keeps position very accurately. Next steps will be to implement ICP odometry, RGBD ICP Odometry, and Visual RGBD odometry.

File: catkin_ws/src/frc_robot/urdf/00-default.urdf.xacro (robot description, xacro)
@@ -52,4 +52,5 @@
     <origin/>
   </xacro:hokuyo_04lx_laser>
+<!--
   <gazebo>
     <plugin name="imu_plugin" filename="libgazebo_ros_imu.so">
@@ -62,4 +63,30 @@
     </plugin>
   </gazebo>
+-->
+  <link name="imu_link"/>
+  <joint name="base_link_to_imu_link" type="fixed">
+    <parent link="base_link"/>
+    <child link="imu_link"/>
+    <origin rpy="0 0 0" xyz="0 0 0"/>
+  </joint>
+  <gazebo reference="imu_link">
+    <gravity>true</gravity>
+    <sensor name="imu_sensor" type="imu">
+      <always_on>true</always_on>
+      <update_rate>100</update_rate>
+      <visualize>true</visualize>
+      <topic>imu</topic>
+      <plugin filename="libgazebo_ros_imu_sensor.so" name="imu_plugin">
+        <topicName>imu</topicName>
+        <bodyName>imu_link</bodyName>
+        <updateRateHZ>50.0</updateRateHZ>
+        <gaussianNoise>0.0</gaussianNoise>
+        <xyzOffset>0 0 0</xyzOffset>
+        <rpyOffset>0 0 0</rpyOffset>
+        <frameName>imu_link</frameName>
+      </plugin>
+      <pose>0 0 0 0 0 0</pose>
+    </sensor>
+  </gazebo>
 <!--                          For Gazebo Simulation                          -->
   <gazebo>
